File: Module-GnuPi/MODUL_GNU-PI_BRIDGE_V100.brd (EAGLE design)
At the start: 56 x 85 mm, 8 parts

Commit message: add many boards
Connections:
- net IO4: now also SV4.11; no longer SV4.12
- net IO8: now also SV4.12; no longer SV4.11
Routing:
- net IO8: track 65.4 -> 71.8 mm
- net IO4: track 84.9 -> 83.2 mm
Other:
- board text added: "+3V3, IO4, SCLK, MOSI, SCL, GPA3, GPA0"
- board text added: "/dev/spidev-0.0"
- board text added: "/dev/spidev-0.1"
- board text added: "GND, IO8, SCK, MISO, SDA, PWM, GPA1"
- board text added: "Module-GnuPi"
- board text removed: "+3V3, IO8, SCLK, MOSI, SCL, GPA3, GPA0"
- board text removed: "GND, IO4, SCK, MISO, SDA, PWM, GPA1"
- board text removed: "for RaspberryPi"
