File: Module-GnuPi/MODUL_GNU-PI_BRIDGE_V100.sch (EAGLE design)
At the start: 8 parts

Commit message: added pdf files
Other:
- note added: "(CC) creative commons 3.0"
- note added: "embedded projects GmbH"
- note removed: "created by Markus Musielak"
Changed lines of the file:
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@@
 <sheet>
 <plain>
-<text x="215.9" y="20.32" size="1.778" layer="91" font="vector">created by Markus Musielak</text>
+<text x="215.9" y="20.32" size="1.778" layer="91" font="vector">embedded projects GmbH</text>
 <wire x1="27.94" y1="66.04" x2="129.54" y2="66.04" width="0.1524" layer="94" style="dashdot"/>
 <wire x1="129.54" y1="66.04" x2="129.54" y2="12.7" width="0.1524" layer="94" style="dashdot"/>
 <text x="71.12" y="10.16" size="1.778" layer="94">Eingang</text>
 <text x="172.72" y="71.12" size="1.778" layer="94">Ausgänge</text>
+<text x="172.72" y="5.08" size="1.778" layer="91" font="vector">(CC) creative commons 3.0</text>
 </plain>
 <instances>
