File: Module-GnuPi/MODUL_GNU-PI_BRIDGE_V1001.sch (EAGLE design)
At the start: 8 parts

Commit message: add many boards
Parts:
- removed U$4: GNUBLINLOGOSIEB, EmbeddedProjectsLogos2:GNUBLINLOGOSIEB
- added U$3: GNUBLINLOGOSIEB, EmbeddedProjectsLogos2:GNUBLINLOGOSIEB
Connections:
- net IO4: now also SV4.11; no longer SV4.12
- net IO8: now also SV4.12; no longer SV4.11
Other:
- note added: "Ausgänge"
- note added: "Eingang"
- note removed: "Input"
- note removed: "Output"
- note removed: "embedded projects GmbH www.gnublin.org Creative Commons 3.0"
Changed lines of the file:
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@@
 <part name="SV5" library="con-ml" deviceset="ML14" device=""/>
 <part name="SV6" library="con-ml" deviceset="ML14" device=""/>
+<part name="GND1" library="supply1" deviceset="GND" device=""/>
 <part name="U$2" library="EmbeddedProjectsLogos2" deviceset="EPLOGO" device="SIEB"/>
-<part name="U$4" library="EmbeddedProjectsLogos2" deviceset="GNUBLINLOGO" device="SIEB"/>
-<part name="GND1" library="supply1" deviceset="GND" device=""/>
+<part name="U$3" library="EmbeddedProjectsLogos2" deviceset="GNUBLINLOGO" device="SIEB"/>
 </parts>
 <sheets>
@@
 <wire x1="27.94" y1="66.04" x2="129.54" y2="66.04" width="0.1524" layer="94" style="dashdot"/>
 <wire x1="129.54" y1="66.04" x2="129.54" y2="12.7" width="0.1524" layer="94" style="dashdot"/>
-<text x="71.12" y="10.16" size="1.778" layer="94">Input</text>
-<text x="172.72" y="71.12" size="1.778" layer="94">Output</text>
-<text x="165.1" y="15.24" size="1.778" layer="91" font="vector">embedded projects GmbH
-www.gnublin.org
-Creative Commons 3.0</text>
+<text x="71.12" y="10.16" size="1.778" layer="94">Eingang</text>
+<text x="172.72" y="71.12" size="1.778" layer="94">Ausgänge</text>
 </plain>
 <instances>
@@
 <instance part="SV5" gate="1" x="185.42" y="111.76"/>
 <instance part="SV6" gate="1" x="223.52" y="111.76"/>
-<instance part="U$2" gate="G$1" x="167.64" y="7.62"/>
-<instance part="U$4" gate="G$1" x="177.8" y="7.62"/>
 <instance part="GND1" gate="1" x="223.52" y="132.08"/>
+<instance part="U$2" gate="G$1" x="170.18" y="12.7"/>
+<instance part="U$3" gate="G$1" x="185.42" y="15.24"/>
 </instances>
 <busses>
@@
 </segment>
 <segment>
-<pinref part="SV4" gate="1" pin="11"/>
-<wire x1="162.56" y1="116.84" x2="154.94" y2="116.84" width="0.1524" layer="91"/>
-<label x="154.94" y="116.84" size="1.27" layer="95"/>
+<pinref part="SV4" gate="1" pin="12"/>
+<wire x1="139.7" y1="116.84" x2="134.62" y2="116.84" width="0.1524" layer="91"/>
+<label x="134.62" y="116.84" size="1.27" layer="95"/>
 </segment>
 </net>
@@
 </segment>
 <segment>
-<pinref part="SV4" gate="1" pin="12"/>
-<wire x1="132.08" y1="116.84" x2="139.7" y2="116.84" width="0.1524" layer="91"/>
-<label x="134.62" y="116.84" size="1.27" layer="95"/>
+<pinref part="SV4" gate="1" pin="11"/>
+<wire x1="154.94" y1="116.84" x2="160.02" y2="116.84" width="0.1524" layer="91"/>
+<label x="154.94" y="116.84" size="1.27" layer="95"/>
 </segment>
 </net>
@@
 </schematic>
 </drawing>
-<compatibility>
-<note version="6.3" minversion="6.2.2" severity="warning">
-Since Version 6.2.2 text objects can contain more than one line,
-which will not be processed correctly with this version.
-</note>
-</compatibility>
 </eagle>

Commit message: added pdf files
Other:
- note added: "(CC) creative commons 3.0"
- note added: "embedded projects GmbH"
- note removed: "created by Markus Musielak"
Changed lines of the file:
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@@
 <sheet>
 <plain>
-<text x="215.9" y="20.32" size="1.778" layer="91" font="vector">created by Markus Musielak</text>
+<text x="215.9" y="20.32" size="1.778" layer="91" font="vector">embedded projects GmbH</text>
 <wire x1="27.94" y1="66.04" x2="129.54" y2="66.04" width="0.1524" layer="94" style="dashdot"/>
 <wire x1="129.54" y1="66.04" x2="129.54" y2="12.7" width="0.1524" layer="94" style="dashdot"/>
 <text x="71.12" y="10.16" size="1.778" layer="94">Eingang</text>
 <text x="172.72" y="71.12" size="1.778" layer="94">Ausgänge</text>
+<text x="175.26" y="5.08" size="1.778" layer="91" font="vector">(CC) creative commons 3.0</text>
 </plain>
 <instances>
