File: Board-EXTENDED/GNUBLIN_EXTENDED_V1_7.sch (EAGLE design)
At the start: 105 parts, among them IC2 AS1324, IC3 AS1324, IC5 A43E26161TSOPII, IC6 LPC313XFET180, IC7 CP21021, IC8 MC78M05ABDT, K1 61001021121, Q4 SX-32 16MHz, U1 DM3D-SF, X1 MINI-USB-32005-201, X2 MINI-USB-32005-201

Commit message: added pdf files
Other:
- note added: "(CC) creative commons 3.0"
Changed lines of the file:
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@@
 <text x="393.1" y="7" size="2.54" layer="94" font="vector">A</text>
 <text x="12.7" y="154.94" size="1.016" layer="94">UART zum Debuggen</text>
+<text x="302" y="6.16" size="1.27" layer="94" font="vector">(CC) creative commons 3.0</text>
 </plain>
 <instances>
@@
 <text x="358.14" y="109.22" size="1.27" layer="94">OTG</text>
 <text x="297.18" y="66.04" size="1.27" layer="94">VCC Select</text>
+<text x="288.4" y="6.26" size="1.27" layer="94" font="vector">(CC) creative commons 3.0</text>
 </plain>
 <instances>
