File: Board-LAN/GNUBLIN_LAN_V2.3.sch (EAGLE design)
At the start: 137 parts, among them IC1 APX803, IC2 AS1324, IC3 AS1324, IC4 CP21021, IC5 A43E26161TSOPII, IC6 LPC313XFET180, IC7 MCP7940SOIC, IC8 MC78M05ABDT, K1 61400416021, K4 G6D-1A-ASI5VDC, Q1 SX-32 - 12 MHz, Q2 BSS123, Q3 32.768kHz, Q4 SX-32 - 25 MHZ, Q5 HC49S - 25MHz, U1 DM3D-SF, U3 ENC28J60-SSOP, X1 J1011F21P, X2 MINI-USB-32005-201

Commit message: added pdf files
Other:
- note added: "(CC) creative commons 3.0"
Changed lines of the file:
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@@
 <text x="393.1" y="7" size="2.54" layer="94" font="vector">A</text>
 <text x="17.78" y="154.94" size="1.016" layer="94">UART zum Debuggen</text>
+<text x="302" y="6.16" size="1.27" layer="94" font="vector">(CC) creative commons 3.0</text>
 </plain>
 <instances>
@@
 <text x="290.46" y="27.84" size="1.778" layer="94">Holzbachstraße 4</text>
 <text x="290.46" y="25.3" size="1.778" layer="94">D-86152 Augsburg</text>
+<text x="288.4" y="6.26" size="1.27" layer="94" font="vector">(CC) creative commons 3.0</text>
 </plain>
 <instances>
