File: Module-CAN/MODUL_CAN_V100.sch (EAGLE design)
At the start: 21 parts, among them IC1 MCP2515-I/SO, IC2 SN65HVD230, Q1 16MHz

Commit message: added pdf files
Other:
- note added: "embedded projects GmbH"
Changed lines of the file:
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@@
 <?xml version="1.0" encoding="utf-8"?>
 <!DOCTYPE eagle SYSTEM "eagle.dtd">
-<eagle version="6.3">
+<eagle version="6.4">
 <drawing>
 <settings>
@@
 <text x="162.56" y="12.7" size="1.778" layer="94" font="vector">Lizenz </text>
 <text x="162.56" y="7.62" size="1.778" layer="94" font="vector">(cc) creative commons 3.0</text>
+<text x="162.56" y="20.32" size="1.778" layer="94" font="vector">embedded projects GmbH</text>
 </plain>
 <instances>
