File: Module-IOExpander/MODUL_PORTEXP_V101.sch (EAGLE design)
At the start: 23 parts, among them IC1 PCA9555D

Commit message: added pdf files
Other:
- note added: "embedded projects GmbH"
Changed lines of the file:
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@@
 <?xml version="1.0" encoding="utf-8"?>
 <!DOCTYPE eagle SYSTEM "eagle.dtd">
-<eagle version="6.3">
+<eagle version="6.4">
 <drawing>
 <settings>
@@
 <text x="167.64" y="12.7" size="1.778" layer="94">Lizenz</text>
 <text x="167.64" y="7.62" size="1.778" layer="94">(CC 3.0) creative commons 3.0</text>
+<text x="167.64" y="20.32" size="1.778" layer="94">embedded projects GmbH</text>
 </plain>
 <instances>
