File: Module-LAN/MODUL_LAN_V102.sch (EAGLE design)
At the start: 30 parts, among them IC1 ENC28J60-SSOP, Q1 CSM-7X-DU, Q4 SX-32 25 MHZ, X1 J1011F21P

Commit message: added pdf files
Other:
- note added: "embedded projects GmbH"
Changed lines of the file:
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@@
 <?xml version="1.0" encoding="utf-8"?>
 <!DOCTYPE eagle SYSTEM "eagle.dtd">
-<eagle version="6.3">
+<eagle version="6.4">
 <drawing>
 <settings>
@@
 <text x="162.56" y="17.78" size="1.778" layer="94" font="vector">created by Markus Musielak</text>
 <text x="162.56" y="12.7" size="1.778" layer="94" font="vector">(CC) creative commons 3.0</text>
+<text x="162.56" y="20.32" size="1.778" layer="94" font="vector">embedded projects GmbH</text>
 </plain>
 <instances>
