File: Module-LM75/MODUL_TEMPERATURE_V100.sch (EAGLE design)
At the start: 19 parts, among them U1 LM75

Commit message: added pdf files
Other:
- note added: "embedded projects GmbH"
Changed lines of the file:
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@@
 <?xml version="1.0" encoding="utf-8"?>
 <!DOCTYPE eagle SYSTEM "eagle.dtd">
-<eagle version="6.3">
+<eagle version="6.4">
 <drawing>
 <settings>
@@
 <wire x1="42.418" y1="137.668" x2="42.418" y2="138.684" width="0.1524" layer="94"/>
 <text x="99.06" y="99.06" size="1.778" layer="91" rot="R180">Term.</text>
-<text x="167.64" y="17.78" size="1.778" layer="94" font="vector">nach www.horter.de</text>
+<text x="177.8" y="15.24" size="1.778" layer="94" font="vector">nach www.horter.de</text>
 <text x="25.146" y="167.386" size="1.778" layer="91">Adressen</text>
 <text x="22.86" y="162.56" size="1.016" layer="91">JP  3  2  1</text>
@@
 <rectangle x1="40.386" y1="157.226" x2="41.656" y2="159.766" layer="94"/>
 <rectangle x1="38.608" y1="159.258" x2="39.878" y2="161.798" layer="94"/>
-<text x="162.56" y="20.32" size="1.778" layer="94" font="vector">created by Markus Musielak</text>
+<text x="162.56" y="17.78" size="1.778" layer="94" font="vector">created by Markus Musielak</text>
 <text x="162.56" y="12.7" size="1.778" layer="94" font="vector">Lizenz</text>
 <text x="162.56" y="7.62" size="1.778" layer="94" font="vector">(CC 3.0) creative commons 3.0</text>
+<text x="162.56" y="20.32" size="1.778" layer="94" font="vector">embedded projects GmbH</text>
 </plain>
 <instances>
